File: hitbox.kicad_pcb (KiCad board)
At the start: 2 copper layers, 5 x 5 mm, 19 parts, among them U1 ER_OLEDM0.91_1x-I2C

Commit message: 邊框與零件位置
Parts:
- moved Home1 103.2 mm to (37.5, 25.7)
- moved Down1 102.8 mm to (67.1, 46.6)
- moved RS1 100.8 mm to (42.0, 25.7)
- moved Start(+)1 99.8 mm to (59.7, 26.2)
- moved U1 99.6 mm to (17.0, 23.5)
- moved LS1 99.3 mm to (46.2, 25.7)
- moved Select(-)1 98.6 mm to (66.2, 26.0)
- moved Left1 96.8 mm to (37.9, 49.3)
- moved Right1 91.8 mm to (95.0, 59.4)
- moved ZL1 89.3 mm to (184.0, 61.0)
- moved A2 86.7 mm to (154.5, 63.2)
- moved ZR1 85.0 mm to (213.9, 63.6)
- moved L1 83.5 mm to (179.2, 31.1)
- moved Y1 81.2 mm to (148.9, 34.1)
- moved R1 79.7 mm to (208.7, 34.1)
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Routing:
- net Net-(A1-GPIO2): track 0.00 -> 68.9 mm
- net Net-(U1-GND): track 0.00 -> 31.9 mm
Other:
- board size 5 x 5 mm -> 218.4 x 118.1 mm

Commit message: 0830佈線
Parts:
- moved A1 27.1 mm to (40.6, 80.0)
- moved U1 18.1 mm to (33.7, 30.5), turned to -90 degrees
- moved Select(-)1 8.49 mm to (59.1, 30.5), turned to 180 degrees
- moved Start(+)1 7.19 mm to (54.0, 30.5), turned to 180 degrees
- moved LS1 5.46 mm to (48.9, 30.5), turned to 180 degrees
- moved RS1 5.11 mm to (43.8, 30.5), turned to 180 degrees
- moved Home1 4.93 mm to (38.7, 30.5), turned to 180 degrees
Routing:
- net Net-(U1-GND): track 31.9 -> 493.8 mm
- net Net-(A1-GPIO12): track 0.00 -> 192.5 mm
- net Net-(A1-GPIO8): track 0.00 -> 181.9 mm
- net Net-(A1-GPIO9): track 0.00 -> 147.9 mm
- net Net-(A1-GPIO13): track 0.00 -> 142.3 mm
- net Net-(A1-GPIO10): track 0.00 -> 123.4 mm
- net Net-(A1-GPIO7): track 0.00 -> 120.5 mm
- net Net-(A1-GPIO6): track 0.00 -> 91.2 mm
- net Net-(A1-GPIO11): track 0.00 -> 88.3 mm
- net Net-(A1-GPIO4): track 0.00 -> 78.0 mm
- net Net-(A1-GPIO1): track 0.00 -> 62.4 mm
- net Net-(A1-GPIO0): track 0.00 -> 62.4 mm
- net Net-(A1-GPIO3): track 0.00 -> 58.0 mm
- net Net-(A1-GPIO20): track 0.00 -> 45.4 mm
- net Net-(A1-GPIO19): track 0.00 -> 44.3 mm
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Other:
- board size 218.4 x 118.1 mm -> 217.2 x 118.1 mm

Commit message: 修改零件位置(未完成)
Parts:
- added REF**: MountingHole_3.2mm_M3, MountingHole:MountingHole_3.2mm_M3, F.Cu at (137.2, 15.2)
- added REF**: MountingHole_3.2mm_M3, MountingHole:MountingHole_3.2mm_M3, F.Cu at (223.5, 15.2)
- added REF**: MountingHole_3.2mm_M3, MountingHole:MountingHole_3.2mm_M3, F.Cu at (142.2, 132.1)
- added REF**: MountingHole_3.2mm_M3, MountingHole:MountingHole_3.2mm_M3, F.Cu at (25.4, 132.1)
- added REF**: MountingHole_3.2mm_M3, MountingHole:MountingHole_3.2mm_M3, F.Cu at (25.4, 15.2)
- added REF**: MountingHole_3.2mm_M3, MountingHole:MountingHole_3.2mm_M3, F.Cu at (223.5, 132.1)
- moved U1 82.2 mm to (99.3, 79.9)
- moved Home1 41.8 mm to (64.4, -2.54)
- moved LS1 41.8 mm to (74.5, -2.54)
- moved RS1 41.8 mm to (69.5, -2.54)
- moved Select(-)1 41.8 mm to (84.7, -2.54)
- moved Start(+)1 41.8 mm to (79.6, -2.54)
- moved A1 6.35 mm to (47.0, 80.0)
Connections:
- U1 pad 1: Net-(U1-GND) -> Net-(A1-GPIO0)
- U1 pad 2: Net-(A1-3V3) -> Net-(A1-GPIO1)
- U1 pad 3: Net-(A1-GPIO1) -> Net-(U1-GND)
- U1 pad 4: Net-(A1-GPIO0) -> Net-(A1-3V3)
Routing:
- net Net-(U1-GND): track 493.8 -> 0.00 mm
- net Net-(A1-GPIO12): track 192.5 -> 0.00 mm
- net Net-(A1-GPIO8): track 181.9 -> 0.00 mm
- net Net-(A1-GPIO9): track 147.9 -> 0.00 mm
- net Net-(A1-GPIO13): track 142.3 -> 0.00 mm
- net Net-(A1-GPIO10): track 123.4 -> 0.00 mm
- net Net-(A1-GPIO7): track 120.5 -> 0.00 mm
- net Net-(A1-GPIO2): track 93.6 -> 0.00 mm
- net Net-(A1-GPIO6): track 91.2 -> 0.00 mm
- net Net-(A1-GPIO4): track 78.0 -> 0.00 mm
- net Net-(A1-GPIO11): track 88.3 -> 11.8 mm
- net Net-(A1-GPIO1): track 62.4 -> 0.00 mm
- net Net-(A1-GPIO0): track 62.4 -> 0.00 mm
- net Net-(A1-GPIO3): track 58.0 -> 0.00 mm
- net Net-(A1-GPIO20): track 45.4 -> 0.00 mm
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Other:
- board size 217.2 x 118.1 mm -> 208.3 x 127 mm

Commit message: 0901更改零件位置
Parts:
- removed the REF** at (137.2, 15.2)
- moved Select(-)1 117.3 mm to (200.7, 15.2)
- moved Start(+)1 102.6 mm to (180.7, 15.2)
- moved LS1 87.9 mm to (160.7, 15.2)
- moved RS1 73.4 mm to (140.7, 15.2)
- moved U1 63.7 mm to (106.3, 16.6)
- moved Home1 59.0 mm to (120.7, 15.2)
- moved A1 56.4 mm to (61.0, 25.4)
- moved L1 17.2 mm to (172.7, 47.0)
- moved R1 16.9 mm to (201.0, 49.1)
- moved Y1 15.9 mm to (144.8, 49.5)
- moved Down1 15.9 mm to (66.9, 62.5)
- moved ZR1 15.9 mm to (205.5, 77.1)
- moved Left1 15.6 mm to (39.0, 64.9)
- moved X1 15.2 mm to (119.4, 61.3)
- moved ZL1 15.0 mm to (177.6, 74.6)
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Connections:
- U1 pad 1: Net-(A1-GPIO0) -> Net-(U1-GND)
- U1 pad 2: Net-(A1-GPIO1) -> Net-(A1-3V3)
- U1 pad 3: Net-(U1-GND) -> Net-(A1-GPIO1)
- U1 pad 4: Net-(A1-3V3) -> Net-(A1-GPIO0)
Routing:
- net Net-(U1-GND): track 0.00 -> 45.7 mm
- net Net-(A1-GPIO11): track 11.8 -> 0.00 mm
- net Net-(A1-GPIO5): track 1.56 -> 0.00 mm
Other:
- outline, holes or cut-outs redrawn

Commit message: 0902佈線
Parts:
- moved LS1 20.0 mm to (140.7, 15.2)
- moved RS1 20.0 mm to (160.7, 15.2)
- moved Select(-)1 20.0 mm to (180.7, 15.2)
- moved Start(+)1 20.0 mm to (200.7, 15.2)
Routing:
- net Net-(U1-GND): track 45.7 -> 800.6 mm
- net Net-(A1-GPIO8): track 0.00 -> 155.8 mm
- net Net-(A1-GPIO12): track 0.00 -> 147.9 mm
- net Net-(A1-GPIO17): track 0.00 -> 124.1 mm
- net Net-(A1-GPIO9): track 0.00 -> 123.6 mm
- net Net-(A1-GPIO19): track 0.00 -> 109.2 mm
- net Net-(A1-GPIO2): track 0.00 -> 109.1 mm
- net Net-(A1-GPIO13): track 0.00 -> 104.5 mm
- net Net-(A1-GPIO7): track 0.00 -> 101.8 mm
- net Net-(A1-GPIO16): track 0.00 -> 100.0 mm
- net Net-(A1-GPIO0): track 0.00 -> 88.4 mm
- net Net-(A1-GPIO10): track 0.00 -> 87.8 mm
- net Net-(A1-GPIO18): track 0.00 -> 86.8 mm
- net Net-(A1-GPIO6): track 0.00 -> 83.9 mm
- net Net-(A1-GPIO1): track 0.00 -> 82.2 mm
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
Commit message: 0903修正按鍵位置及增加標示文字
Parts:
- moved X1 28.0 mm to (144.8, 49.5)
- moved Y1 28.0 mm to (119.4, 61.3)
- moved REF** 15.2 mm to (127.0, 132.1)
- renumbered Start(+)1 to +, Select(-)1 to -, Home1 to Home, LS1 to LS, RS1 to RS
Routing:
- net Net-(U1-GND): track 800.6 -> 718.7 mm
- net Net-(A1-GPIO11): track 52.4 -> 85.3 mm
- net Net-(A1-GPIO10): track 87.8 -> 54.9 mm
Other:
- outline, holes or cut-outs redrawn
- board text added: "A"
- board text added: "B"
- board text added: "L"
- board text added: "R"
- board text added: "X"
- board text added: "Y"
- board text added: "ZL"
- board text added: "ZR"
- board text added: "←"
- board text added: "↑"
- board text added: "→"
- board text added: "↓"

Commit message: 0904修正走線
Connections:
- net Net-(U1-GND) renamed GND
Routing:
- net Net-(A1-3V3): track 52.5 -> 169.2 mm
- net GND: track 718.7 -> 791.1 mm
- net Net-(A1-GPIO17): track 124.1 -> 143.9 mm
- net Net-(A1-GPIO16): track 100.0 -> 118.9 mm
- net Net-(A1-GPIO12): track 147.9 -> 137.0 mm
- net Net-(A1-GPIO5): track 49.3 -> 51.2 mm
- net Net-(A1-GPIO11): track 85.3 -> 86.2 mm
- added copper zone on B.Cu, net (none)
- added copper zone on F.Cu, net (none)
- added copper zone on F.Cu, net GND
