File: hitbox.kicad_pcb (KiCad board)
At the start: 2 copper layers, 208.3 x 127 mm, 24 parts, among them U1 ER_OLEDM0.91_1x-I2C

Commit message: 0906_1.0
Parts:
- moved A2 6.94 mm to (142.7, 77.0)
- moved B1 6.94 mm to (117.4, 88.8)
- moved ZL1 6.94 mm to (170.6, 74.6)
- moved ZR1 6.94 mm to (198.5, 77.0)
Routing:
- net GND: track 791.1 -> 811.9 mm
- net Net-(A1-GPIO7): track 101.8 -> 94.9 mm
- net Net-(A1-GPIO6): track 83.9 -> 77.2 mm
- net Net-(A1-GPIO8): track 155.8 -> 149.3 mm
- net Net-(A1-GPIO9): track 123.6 -> 117.1 mm
- added copper zone on B.Cu, net GND
- removed copper zone on B.Cu, net (none)
- removed copper zone on F.Cu, net (none)

Commit message: 0907修改走線
Routing:
- net Net-(A1-3V3): track 169.2 -> 191.5 mm
- net Net-(A1-GPIO17): track 143.9 -> 150.4 mm
- net Net-(A1-GPIO10): track 54.9 -> 57.8 mm
- net Net-(A1-GPIO12): track 137.0 -> 139.4 mm
- net GND: track 811.9 -> 814.3 mm
- net Net-(A1-GPIO13): track 104.5 -> 106.7 mm
- net Net-(A1-GPIO11): track 86.2 -> 87.9 mm
- net Net-(A1-GPIO7): track 94.9 -> 96.5 mm
- net Net-(A1-GPIO6): track 77.2 -> 78.8 mm
- net Net-(A1-GPIO16): track 118.9 -> 120.4 mm
- net Net-(A1-GPIO8): track 149.3 -> 150.1 mm
- net Net-(A1-GPIO9): track 117.1 -> 117.9 mm

Commit message: 0911修改GND線路
Routing:
- net GND: track 814.3 -> 905.3 mm
- net Net-(A1-3V3): track 191.5 -> 195.8 mm
- net Net-(A1-GPIO5): track 51.2 -> 55.1 mm
- net Net-(A1-GPIO19): track 109.2 -> 111.2 mm

Commit message: 0929_3dmodel
Other:
- board text added: "2026/09/14"
Changed lines of the file:
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@@
 		(tags "Through hole pin header THT 1x02 2.54mm single row")
 		(property "Reference" "-"
-			(at -17.46 -15.24 180)
+			(at -10.216 -17.272 180)
 			(layer "F.SilkS")
 			(effects
@@
 		(tags "Through hole pin header THT 1x02 2.54mm single row")
 		(property "Reference" "+"
-			(at -17.78 -15.24 180)
+			(at -10.216 -17.272 180)
 			(layer "F.SilkS")
 			(effects
@@
 		(tags "Through hole pin header THT 1x02 2.54mm single row")
 		(property "Reference" "LS"
-			(at -16.82 -15.24 180)
+			(at -10.216 -17.272 180)
 			(layer "F.SilkS")
 			(effects
@@
 		(tags "Through hole pin header THT 1x02 2.54mm single row")
 		(property "Reference" "Home"
-			(at -19.548 -15.24 180)
+			(at -10.216 -17.272 180)
 			(layer "F.SilkS")
 			(effects
@@
 		(tags "Through hole pin header THT 1x02 2.54mm single row")
 		(property "Reference" "RS"
-			(at -17.14 -15.24 180)
+			(at -10.216 -17.272 180)
 			(layer "F.SilkS")
 			(effects
@@
 		(layer "Edge.Cuts")
 	)
+	(gr_text "2026/09/14"
+		(at 209.296 134.874 0)
+		(layer "F.SilkS")
+		(effects
+			(font
+				(size 1 1)
+				(thickness 0.1)
+			)
+			(justify left bottom)
+		)
+	)
 	(gr_text "B"
